Commit message: 将gazebo中机器人模型固定到地面并修改机器人关节控制模式

File: src/pkg_ur10e_gripper_moveit/config/gazebo_ur10e_with_robotiq_2f_85.urdf (robot description, URDF)
Before this commit: robot ur10e_with_robotiq_2f_85, 20 links, 19 joints
Links:
- added link world
Joints:
- added joint world_base_joint: type fixed, parent world, child base_link, origin xyz=0 0 0 rpy=0 0 0
